File: ghost/ghost.kicad_pcb (KiCad board)
At the start: 2 copper layers, 185 x 52 mm, 60 parts, among them J1 TC2030-IDC, J2 USB_B, K0 K00, K1 K00, K10 K00, K11 K00, K12 K00, K13 K00, K14 K00, K15 K00, K16 K00, K17 K00, K18 K00, K19 K00, K2 K00, K20 K00, K21 K00, K22 K00, K23 K00, K24 K00, K25 K00, K26 K00, K27 K00, K28 K00, K29 K00, K3 K00, K4 K00, K5 K00, K6 K00, K7 K00, K8 K00, K9 K00, U1 MIC550X, U2 ATXMEGA-A4U-EPAD

Commit message: add spectre
Parts:
- removed OSHW_Logo: G***, logo:OSHW_5x5mm_SilkS
- added ?: , logo:OSHW_3x3mm_SilkS, B.Cu at (35.5, 48.8)
Other:
- outline, holes or cut-outs redrawn
- board text added: "jem@seethis.link"
- board text added: "v1"
- board text removed: "v1 2018 jem@seethis.link"
